File: Guitar-ToneFenderTB.kicad_pcb (KiCad board)
At the start: 2 copper layers, 53 x 35 mm, 15 parts, among them J1 Screw_Terminal_1x02, J2 Screw_Terminal_1x02, J3 Screw_Terminal_1x01

Commit message: Updated silkscreen text with C2 5mm spacing, and PCBWay product number code
Parts:
- moved G*** 2.00 mm to (189.5, 117.0)
Other:
- board text added: "5mm radial"
- board text added: "Fender Bass Treble tonestack v 1.0.0 Ian Evans 08/07/2025 github.com/shampeon/Guitar-ToneFenderTB WayWayWay"
- board text removed: "Fender Bass Treble tonestack v 1.0.0 Ian Evans 08/07/2025 github.com/shampeon/Guitar-ToneFenderTB"
Changed lines of the file:
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@@
 	(footprint "LOGO"
 		(layer "F.Cu")
-		(at 189.5 115)
+		(at 189.5 117)
 		(property "Reference" "G***"
 			(at 0 0 0)
@@
 		)
 	)
+	(gr_text "5mm radial"
+		(at 172.5 117.5 90)
+		(layer "F.SilkS")
+		(effects
+			(font
+				(size 1 1)
+				(thickness 0.15)
+			)
+			(justify left bottom)
+		)
+	)
 	(gr_text "Treble"
 		(at 197 122.1 0)
@@
 		)
 	)
-	(gr_text "Fender Bass Treble tonestack\nv 1.0.0\nIan Evans\n08/07/2025\ngithub.com/shampeon/Guitar-ToneFenderTB"
+	(gr_text "Fender Bass Treble tonestack\nv 1.0.0\nIan Evans\n08/07/2025\ngithub.com/shampeon/Guitar-ToneFenderTB\nWayWayWay"
 		(at 194.5 109.5 0)
 		(layer "B.SilkS")
