File: Guitar-ToneFenderTB.kicad_sch (KiCad schematic)
At the start: 12 parts, among them J1 Screw_Terminal_1x02, J2 Screw_Terminal_1x02, J3 Screw_Terminal_1x01

Commit message: Fixed error in schematic, enlarged through holes for caps.
Parts:
- C2: footprint Capacitor_THT:C_Axial_L22.0mm_D9.5mm_P27.50mm_Horizontal -> Local:C_Axial_L22.0mm_D9.5mm_P27.50mm_Horizontal
- C3: footprint Capacitor_THT:C_Axial_L12.0mm_D6.5mm_P15.00mm_Horizontal -> Local:C_Axial_L12.0mm_D6.5mm_P15.00mm_Horizontal
Connections:
- net at R1.1: now also C1.1, J1.2
Changed lines of the file:
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@@
+	)
+	(junction
+		(at 88.9 54.61)
+		(diameter 0)
+		(color 0 0 0 0)
 	)
 	(junction
@@
 	(wire
 		(pts
-			(xy 71.12 54.61) (xy 93.98 54.61)
+			(xy 71.12 54.61) (xy 88.9 54.61)
+		)
+		(stroke
+			(width 0)
+			(type default)
+		)
+	)
+	(wire
+		(pts
+			(xy 88.9 54.61) (xy 88.9 57.15)
 		)
 		(stroke
@@
 	(wire
 		(pts
-			(xy 88.9 54.356) (xy 88.9 57.15)
-		)
-		(stroke
-			(width 0)
-			(type default)
-		)
-	)
-	(wire
-		(pts
 			(xy 71.12 59.69) (xy 71.12 60.706)
 		)
@@
 		(pts
 			(xy 101.6 54.61) (xy 111.76 54.61)
+		)
+		(stroke
+			(width 0)
+			(type default)
+		)
+	)
+	(wire
+		(pts
+			(xy 88.9 54.61) (xy 93.98 54.61)
 		)
 		(stroke
@@
 			)
 		)
-		(property "Footprint" "Capacitor_THT:C_Axial_L12.0mm_D6.5mm_P15.00mm_Horizontal"
+		(property "Footprint" "Local:C_Axial_L12.0mm_D6.5mm_P15.00mm_Horizontal"
 			(at 101.6 81.5848 0)
 			(effects
@@
 			)
 		)
-		(property "Footprint" "Capacitor_THT:C_Axial_L22.0mm_D9.5mm_P27.50mm_Horizontal"
+		(property "Footprint" "Local:C_Axial_L22.0mm_D9.5mm_P27.50mm_Horizontal"
 			(at 93.98 70.8152 0)
 			(effects
